File: 2063-Z80.kicad_pcb (KiCad board)
At the start: 4 copper layers, 100 x 100 mm, 84 parts, among them J1 Conn_01x05, J10 Conn_01x07, J11 Conn_02x03, J12 Conn_01x02, J2 DM3D-SF(41), J3 Conn_02x20, J4 Conn_02x05, J5 Conn_02x05, J6 0548190519, J7 Conn_02x13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

Commit message: dd net ties to U3 for EZ-hacking
Parts:
- added NT1: Net-Tie_2, NetTie:NetTie-2_SMD_Pad0.5mm, B.Cu at (161.2, 63.0)
- added NT2: Net-Tie_2, NetTie:NetTie-2_SMD_Pad0.5mm, B.Cu at (146.8, 57.0)
Routing:
- net GND: track 9.70 -> 11.2 mm
Changed lines of the file:
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@@
     (thickness 1.6)
     (drawings 113)
-    (tracks 2238)
+    (tracks 2241)
     (zones 0)
-    (modules 84)
+    (modules 86)
     (nets 153)
   )
@@
   (net 148 "Net-(U5-Pad17)")
   (net 149 /~DTRB)
-  (net 150 "Net-(U3-Pad30)")
-  (net 151 "Net-(U3-Pad1)")
-  (net 152 "Net-(J12-Pad2)")
+  (net 150 "Net-(J12-Pad2)")
+  (net 151 "Net-(NT1-Pad2)")
+  (net 152 "Net-(NT2-Pad2)")
   (net_class Default "This is the default net class."
     (clearance 0.1524)
@@
     (add_net "Net-(J6-Pad3)")
     (add_net "Net-(J6-Pad4)")
+    (add_net "Net-(NT1-Pad2)")
+    (add_net "Net-(NT2-Pad2)")
     (add_net "Net-(Q1-Pad2)")
     (add_net "Net-(R12-Pad1)")
     (add_net "Net-(R13-Pad1)")
     (add_net "Net-(S1-Pad1)")
-    (add_net "Net-(U3-Pad1)")
-    (add_net "Net-(U3-Pad30)")
     (add_net "Net-(U4-Pad7)")
     (add_net "Net-(U5-Pad10)")
@@
     (add_net "Net-(X2-Pad1)")
   )
+  (module NetTie:NetTie-2_SMD_Pad0.5mm (layer B.Cu)
+    (at 146.8 56.95 270)
+    (descr "Net tie, 2 pin, 0.5mm square SMD pads")
+    (tags "net tie")
+    (attr virtual)
+    (fp_text reference NT2 (at 0 1.2 270) (layer B.SilkS) hide
+      (effects (font (size 1 1) (thickness 0.15)) (justify mirror))
+    )
+    (fp_text value Net-Tie_2 (at 0 -1.2 270) (layer B.Fab)
+      (effects (font (size 1 1) (thickness 0.15)) (justify mirror))
+    )
+    (fp_line (start -1 0.5) (end -1 -0.5) (layer B.CrtYd) (width 0.05))
+    (fp_line (start -1 -0.5) (end 1 -0.5) (layer B.CrtYd) (width 0.05))
+    (fp_line (start 1 -0.5) (end 1 0.5) (layer B.CrtYd) (width 0.05))
+    (fp_line (start 1 0.5) (end -1 0.5) (layer B.CrtYd) (width 0.05))
+    (fp_poly (pts (xy -0.5 0.25) (xy 0.5 0.25) (xy 0.5 -0.25) (xy -0.5 -0.25)) (layer B.Cu) (width 0))
+    (pad 2 smd circle (at 0.5 0 270) (size 0.5 0.5) (layers B.Cu)
+      (net 152 "Net-(NT2-Pad2)"))
+    (pad 1 smd circle (at -0.5 0 270) (size 0.5 0.5) (layers B.Cu)
+      (net 14 GND))
+  )
+  (module NetTie:NetTie-2_SMD_Pad0.5mm (layer B.Cu)
+    (at 161.2 63)
+    (descr "Net tie, 2 pin, 0.5mm square SMD pads")
+    (tags "net tie")
+    (attr virtual)
+    (fp_text reference NT1 (at 0 1.2) (layer B.SilkS) hide
+      (effects (font (size 1 1) (thickness 0.15)) (justify mirror))
+    )
+    (fp_text value Net-Tie_2 (at 0 -1.2) (layer B.Fab)
+      (effects (font (size 1 1) (thickness 0.15)) (justify mirror))
+    )
+    (fp_line (start -1 0.5) (end -1 -0.5) (layer B.CrtYd) (width 0.05))
+    (fp_line (start -1 -0.5) (end 1 -0.5) (layer B.CrtYd) (width 0.05))
+    (fp_line (start 1 -0.5) (end 1 0.5) (layer B.CrtYd) (width 0.05))
+    (fp_line (start 1 0.5) (end -1 0.5) (layer B.CrtYd) (width 0.05))
+    (fp_poly (pts (xy -0.5 0.25) (xy 0.5 0.25) (xy 0.5 -0.25) (xy -0.5 -0.25)) (layer B.Cu) (width 0))
+    (pad 2 smd circle (at 0.5 0) (size 0.5 0.5) (layers B.Cu)
+      (net 151 "Net-(NT1-Pad2)"))
+    (pad 1 smd circle (at -0.5 0) (size 0.5 0.5) (layers B.Cu)
+      (net 14 GND))
+  )
   (module Resistor_THT:R_Axial_DIN0204_L3.6mm_D1.6mm_P5.08mm_Horizontal (layer F.Cu)
     (at 171.16044 55.19166)
@@
     (fp_line (start 0.74 -0.8) (end 0.74 0.8) (layer F.Fab) (width 0.1))
     (pad 2 thru_hole oval (at 5.08 0) (size 1.4 1.4) (drill 0.7) (layers *.Cu *.Mask)
-      (net 152 "Net-(J12-Pad2)"))
+      (net 150 "Net-(J12-Pad2)"))
     (pad 1 thru_hole circle (at 0 0) (size 1.4 1.4) (drill 0.7) (layers *.Cu *.Mask)
       (net 14 GND))
@@
     (fp_line (start -0.635 -1.27) (end 1.27 -1.27) (layer F.Fab) (width 0.1))
     (pad 2 thru_hole oval (at 0 2.54) (size 1.7 1.7) (drill 1) (layers *.Cu *.Mask)
-      (net 152 "Net-(J12-Pad2)"))
+      (net 150 "Net-(J12-Pad2)"))
     (pad 1 thru_hole rect (at 0 0) (size 1.7 1.7) (drill 1) (layers *.Cu *.Mask)
       (net 23 +5V))
@@
       (net 39 /D2))
     (pad 30 thru_hole oval (at 15.24 5.08) (size 1.6 1.6) (drill 0.8) (layers *.Cu *.Mask)
-      (net 150 "Net-(U3-Pad30)"))
+      (net 151 "Net-(NT1-Pad2)"))
     (pad 14 thru_hole oval (at 0 33.02) (size 1.6 1.6) (drill 0.8) (layers *.Cu *.Mask)
       (net 33 /D1))
@@
       (net 46 /D4))
     (pad 2 thru_hole oval (at 0 2.54) (size 1.6 1.6) (drill 0.8) (layers *.Cu *.Mask)
-      (net 152 "Net-(J12-Pad2)"))
+      (net 150 "Net-(J12-Pad2)"))
     (pad 17 thru_hole oval (at 15.24 38.1) (size 1.6 1.6) (drill 0.8) (layers *.Cu *.Mask)
       (net 44 /D3))
     (pad 1 thru_hole rect (at 0 0) (size 1.6 1.6) (drill 0.8) (layers *.Cu *.Mask)
-      (net 151 "Net-(U3-Pad1)"))
+      (net 152 "Net-(NT2-Pad2)"))
     (model ${KISYS3DMOD}/Package_DIP.3dshapes/DIP-32_W15.24mm_Socket.wrl
       (at (xyz 0 0 0))
@@
   (via (at 178.45278 86.28888) (size 0.8) (drill 0.45) (layers F.Cu B.Cu) (net 14))
   (via (at 184.41416 106.09834) (size 0.8) (drill 0.45) (layers F.Cu B.Cu) (net 14))
+  (segment (start 160.7 63) (end 160.2 63) (width 0.5) (layer B.Cu) (net 14))
+  (segment (start 146.8 55.5) (end 146.85 55.45) (width 0.5) (layer B.Cu) (net 14))
+  (segment (start 146.8 56.45) (end 146.8 55.5) (width 0.5) (layer B.Cu) (net 14))
   (via (at 193.9798 126.238) (size 0.8) (drill 0.45) (layers F.Cu B.Cu) (net 15))
   (segment (start 190.5 126.238) (end 193.9798 126.238) (width 0.1524) (layer F.Cu) (net 15))
@@
   (segment (start 195.98386 97.79254) (end 195.89242 97.88398) (width 0.1524) (layer B.Cu) (net 149))
   (segment (start 195.98386 96.01962) (end 195.98386 97.79254) (width 0.1524) (layer B.Cu) (net 149))
-  (via (at 136.40816 59.2836) (size 0.8) (drill 0.45) (layers F.Cu B.Cu) (net 152))
-  (segment (start 136.3218 59.19724) (end 136.40816 59.2836) (width 0.1524) (layer B.Cu) (net 152))
-  (segment (start 136.3218 55.30596) (end 136.3218 59.19724) (width 0.1524) (layer B.Cu) (net 152))
-  (segment (start 145.6436 59.2836) (end 146.812 60.452) (width 0.1524) (layer F.Cu) (net 152))
-  (segment (start 136.40816 59.2836) (end 145.6436 59.2836) (width 0.1524) (layer F.Cu) (net 152))
-  (segment (start 147.611999 61.251999) (end 154.028039 61.251999) (width 0.1524) (layer F.Cu) (net 152))
-  (segment (start 146.812 60.452) (end 147.611999 61.251999) (width 0.1524) (layer F.Cu) (net 152))
-  (via (at 154.028039 61.251999) (size 0.8) (drill 0.45) (layers F.Cu B.Cu) (net 152))
-  (segment (start 154.028039 61.251999) (end 154.028039 55.295901) (width 0.1524) (layer B.Cu) (net 152))
-  (segment (start 154.76728 54.55666) (end 156.6418 54.55666) (width 0.1524) (layer B.Cu) (net 152))
-  (segment (start 154.028039 55.295901) (end 154.76728 54.55666) (width 0.1524) (layer B.Cu) (net 152))
+  (via (at 136.40816 59.2836) (size 0.8) (drill 0.45) (layers F.Cu B.Cu) (net 150))
+  (segment (start 136.3218 59.19724) (end 136.40816 59.2836) (width 0.1524) (layer B.Cu) (net 150))
+  (segment (start 136.3218 55.30596) (end 136.3218 59.19724) (width 0.1524) (layer B.Cu) (net 150))
+  (segment (start 145.6436 59.2836) (end 146.812 60.452) (width 0.1524) (layer F.Cu) (net 150))
+  (segment (start 136.40816 59.2836) (end 145.6436 59.2836) (width 0.1524) (layer F.Cu) (net 150))
+  (segment (start 147.611999 61.251999) (end 154.028039 61.251999) (width 0.1524) (layer F.Cu) (net 150))
+  (segment (start 146.812 60.452) (end 147.611999 61.251999) (width 0.1524) (layer F.Cu) (net 150))
+  (via (at 154.028039 61.251999) (size 0.8) (drill 0.45) (layers F.Cu B.Cu) (net 150))
+  (segment (start 154.028039 61.251999) (end 154.028039 55.295901) (width 0.1524) (layer B.Cu) (net 150))
+  (segment (start 154.76728 54.55666) (end 156.6418 54.55666) (width 0.1524) (layer B.Cu) (net 150))
+  (segment (start 154.028039 55.295901) (end 154.76728 54.55666) (width 0.1524) (layer B.Cu) (net 150))
   (zone (net 14) (net_name GND) (layer In1.Cu) (hatch edge 0.508)
     (connect_pads yes (clearance 0.2032))
