File: 2063-Z80.kicad_pcb (KiCad board)
At the start: 4 copper layers, 100 x 100 mm, 94 parts, among them J1 Conn_01x05, J10 Conn_01x07, J11 Conn_02x03, J12 Conn_01x02, J13 Conn_01x06, J14 Conn_01x02, J2 DM3D-SF(41), J3 Conn_02x20, J4 Conn_02x05, J5 Conn_02x05, J6 0548190519, J7 Conn_02x13, J8 Conn_01x05, J9 Conn_01x02, Q1 PN2222, U1 Z80-CPU, U10 74HC32, U11 74HCT132, U12 ICL3232CPZ, U13 74HC32, U2 AS6C4008-55PCN, U20 LM1117-3.3, U3 SST39SF010, U4 Z80-CTC, U5 Z80-SIO-0, U6 74HC374, U7 74HC374, U8 74LS244, U9 74HC138, X1 ACH-10.000MHZ-EK, X2 ECS-2100A-018

Commit message: Merge version 4.3 into main
Parts:
- removed J13: Conn_01x06, Connector_PinHeader_2.54mm:PinHeader_1x06_P2.54mm_Horizontal
- removed J14: Conn_01x02, Connector_PinHeader_2.54mm:PinHeader_1x02_P2.54mm_Horizontal
- removed R17, R21, R22: 100K, Resistor_THT:R_Axial_DIN0204_L3.6mm_D1.6mm_P5.08mm_Horizontal
- removed R18, R19, R20: 2K7, Resistor_THT:R_Axial_DIN0204_L3.6mm_D1.6mm_P5.08mm_Horizontal
Connections:
- U5 pad 17: /SIO_RTSA -> Net-(U5-Pad17)
Routing:
- net /SIO_RXA: track 117.4 -> 54.7 mm, vias 5 -> 2
- net /SIO_RTSA: track 54.4 -> 0.00 mm, vias 1 -> 0
- net /SIO_RXB: track 91.9 -> 46.3 mm, vias 1 -> 0
- net /SIO_TXA: track 74.0 -> 51.6 mm, vias 5 -> 2
- net Net-(J13-Pad3): track 18.8 -> 0.00 mm
- net Net-(J13-Pad5): track 6.63 -> 0.00 mm
- net Net-(J13-Pad4): track 3.11 -> 0.00 mm
- net +5V: track 43.4 -> 40.8 mm, vias 6 -> 4
- net /USER1: track 38.2 -> 35.8 mm
- net Net-(J13-Pad2): track 2.12 -> 0.00 mm
- net /SIO_CLKB: track 28.7 -> 30.6 mm
- net /SIO_CLKA: track 19.3 -> 20.9 mm
- net /PRN_D7: track 43.2 -> 42.3 mm
- net GND: vias 24 -> 20
Other:
- board text added: "74HC138"
- board text added: "74HC32"
- board text added: "74HC374"
- board text added: "74LS244"
- board text added: "Rev 2063.4.3"
- board text removed: "'138"
- board text removed: "'244"
- board text removed: "'32"
- board text removed: "'374"
- board text removed: "100K"
- board text removed: "2063.4.2"
- board text removed: "Rev 2063.4.2"

Commit message: Change teh silkscreen label on U2 to AS6C4008
Other:
- board text added: "AS6C4008 SRAM"
Changed lines of the file:
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@@
     (effects (font (size 1 1) (thickness 0.15)))
   )
-  (gr_text "AS6C1008\nSRAM" (at 136.144 64.008) (layer F.SilkS)
+  (gr_text "AS6C4008\nSRAM" (at 136.144 64.008) (layer F.SilkS)
     (effects (font (size 1 1) (thickness 0.15)))
   )

Commit message: Change U2 label on back silkscreen.
Other:
- board text removed: "AS6C1008 SRAM"
Changed lines of the file:
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@@
     (effects (font (size 1 1) (thickness 0.15)) (justify mirror))
   )
-  (gr_text "AS6C1008\nSRAM" (at 134.62 67.564) (layer B.SilkS)
+  (gr_text "AS6C4008\nSRAM" (at 134.62 67.564) (layer B.SilkS)
     (effects (font (size 1 1) (thickness 0.15)) (justify mirror))
   )

Commit message: Change the rev number in the silks too
Other:
- board text added: "Rev 2063.4.3.1"
- board text removed: "Rev 2063.4.3"
Changed lines of the file:
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@@
     (effects (font (size 1.016 1.016) (thickness 0.2286)))
   )
-  (gr_text "Rev 2063.4.3" (at 171.196 52.2986) (layer B.SilkS)
+  (gr_text "Rev 2063.4.3.1" (at 171.196 52.2986) (layer B.SilkS)
     (effects (font (size 1 1) (thickness 0.15)) (justify mirror))
   )
-  (gr_text "Rev 2063.4.3" (at 182.8038 52.0192) (layer F.SilkS)
+  (gr_text "Rev 2063.4.3.1" (at 182.8038 52.0192) (layer F.SilkS)
     (effects (font (size 1 1) (thickness 0.15)))
   )
